File: bluetooth.sch (KiCad schematic (older format))
At the start: 58 parts, among them P100 LIPO, P110 CONN_1, P111 CONN_1, P112 CONN_1, P113 CONN_1, P114 CONN_1, P115 CONN_1, P12 CONN_1, P13 CONN_1, P14 CONN_1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

Commit message: Import into KiCAD 5
Parts:
- C11, C14, C16, C18: symbol C -> HHKB_controller-rescue:C
- C12, C15: symbol CAPAPOL -> HHKB_controller-rescue:CAPAPOL
- D10, D4: symbol LED -> HHKB_controller-rescue:LED
- D11, D2: symbol DIODESCH -> HHKB_controller-rescue:DIODESCH
- D3, D9: symbol LED_DUAL -> HHKB_controller-rescue:LED_DUAL
- D5: symbol D -> HHKB_controller-rescue:D
- L1: symbol INDUCTOR_SMALL -> HHKB_controller-rescue:INDUCTOR_SMALL
- P100: symbol CONN_2 -> HHKB_controller-rescue:CONN_2
- P110, P111, P112, P113, P114, P115, P12, P13, P14, P15: symbol CONN_1 -> HHKB_controller-rescue:CONN_1
- Q1, Q10, Q3: symbol MOSFET_N -> HHKB_controller-rescue:MOSFET_N
- Q4: symbol MOSFET_P -> HHKB_controller-rescue:MOSFET_P
- Q5: symbol MOS_P -> HHKB_controller-rescue:MOS_P
- R1, R10, R11, R12, R13, R14, R16, R17, R18, R19, R20, R21, R22, R23, R24, R25, R26, R27, R30, R6, R7, R8, R9: symbol R -> HHKB_controller-rescue:R
- SW2: symbol SW_DPDT -> HHKB_controller-rescue:SW_DPDT
- U2: symbol LDO_REGULATOR -> HHKB_controller-rescue:LDO_REGULATOR
- U3: symbol HT7750A -> HHKB_controller-rescue:HT7750A
- U4: symbol LTC4054 -> HHKB_controller-rescue:LTC4054
- U5: symbol RN42 -> HHKB_controller-rescue:RN42
